File: 02_Batt_Alim.sch (KiCad schematic (older format))
At the start: 31 parts, among them IC1 TP4056, J1 Conn_01x01, J2 Conn_01x01, J3 Conn_01x01, J4 Conn_01x01, J5 Conn_01x01, J6 Conn_01x01, J9 Conn_01x01, U1 ME2108A50M3

Commit message: changed to new library
Parts:
- IC1: footprint Chimere:SOP-8 -> Chimere_comps:SOP-8; symbol Chimere:TP4056 -> Chimere_comps:TP4056
- U1: symbol Chimere:ME2108A50M3 -> Chimere_comps:ME2108A50M3
Changed lines of the file:
@@
 GND
 $Comp
-L Chimere:TP4056 IC1
+L Chimere_comps:TP4056 IC1
 U 1 1 5FD80F7F
 P 2750 2625
 F 0 "IC1" H 2750 3192 50  0000 C CNN
 F 1 "TP4056" H 2750 3101 50  0000 C CNN
-F 2 "Chimere:SOP-8" H 2750 2625 50  0001 L BNN
+F 2 "Chimere_comps:SOP-8" H 2750 2625 50  0001 L BNN
 F 3 "C16581" H 2750 2625 50  0001 L BNN
 	1    2750 2625
@@
 	2300 4250 2300 3900
 $Comp
-L Chimere:ME2108A50M3 U1
+L Chimere_comps:ME2108A50M3 U1
 U 1 1 5FD912E5
 P 8075 4450

Commit message: changement librairie Chimère split
Parts:
- J1, J2, J3, J4, J5, J6, J9: footprint Chimere:Castellated_conn -> Chimere_mods:Castellated_conn
- L1: footprint Chimere:L_Sunlord_MWSA0603S_6.6x7.0x2.8mm -> Chimere_comps:L_Sunlord_MWSA0603S_6.6x7.0x2.8mm
Changed lines of the file:
@@
 F 0 "J1" H 9880 4192 50  0000 L CNN
 F 1 "Conn_01x01" H 9880 4101 50  0000 L CNN
-F 2 "Chimere:Castellated_conn" H 9800 4150 50  0001 C CNN
+F 2 "Chimere_mods:Castellated_conn" H 9800 4150 50  0001 C CNN
 F 3 "~" H 9800 4150 50  0001 C CNN
 	1    9800 4150
@@
 F 0 "J2" H 9880 4367 50  0000 L CNN
 F 1 "Conn_01x01" H 9880 4276 50  0000 L CNN
-F 2 "Chimere:Castellated_conn" H 9800 4325 50  0001 C CNN
+F 2 "Chimere_mods:Castellated_conn" H 9800 4325 50  0001 C CNN
 F 3 "~" H 9800 4325 50  0001 C CNN
 	1    9800 4325
@@
 F 0 "J3" H 9880 5492 50  0000 L CNN
 F 1 "Conn_01x01" H 9880 5401 50  0000 L CNN
-F 2 "Chimere:Castellated_conn" H 9800 5450 50  0001 C CNN
+F 2 "Chimere_mods:Castellated_conn" H 9800 5450 50  0001 C CNN
 F 3 "~" H 9800 5450 50  0001 C CNN
 	1    9800 5450
@@
 F 0 "J9" H 9880 4567 50  0000 L CNN
 F 1 "Conn_01x01" H 9880 4476 50  0000 L CNN
-F 2 "Chimere:Castellated_conn" H 9800 4525 50  0001 C CNN
+F 2 "Chimere_mods:Castellated_conn" H 9800 4525 50  0001 C CNN
 F 3 "~" H 9800 4525 50  0001 C CNN
 	1    9800 4525
@@
 F 0 "J6" H 9880 5317 50  0000 L CNN
 F 1 "Conn_01x01" H 9880 5226 50  0000 L CNN
-F 2 "Chimere:Castellated_conn" H 9800 5275 50  0001 C CNN
+F 2 "Chimere_mods:Castellated_conn" H 9800 5275 50  0001 C CNN
 F 3 "~" H 9800 5275 50  0001 C CNN
 	1    9800 5275
@@
 F 0 "J5" H 9880 5117 50  0000 L CNN
 F 1 "Conn_01x01" H 9880 5026 50  0000 L CNN
-F 2 "Chimere:Castellated_conn" H 9800 5075 50  0001 C CNN
+F 2 "Chimere_mods:Castellated_conn" H 9800 5075 50  0001 C CNN
 F 3 "~" H 9800 5075 50  0001 C CNN
 	1    9800 5075
@@
 F 0 "J4" H 9880 4817 50  0000 L CNN
 F 1 "Conn_01x01" H 9880 4726 50  0000 L CNN
-F 2 "Chimere:Castellated_conn" H 9800 4775 50  0001 C CNN
+F 2 "Chimere_mods:Castellated_conn" H 9800 4775 50  0001 C CNN
 F 3 "~" H 9800 4775 50  0001 C CNN
 	1    9800 4775
@@
 F 0 "L1" V 7369 3500 50  0000 C CNN
 F 1 "MWSA0603S-330MT" V 7650 3500 50  0000 C CNN
-F 2 "Chimere:L_Sunlord_MWSA0603S_6.6x7.0x2.8mm" H 7550 3500 50  0001 C CNN
+F 2 "Chimere_comps:L_Sunlord_MWSA0603S_6.6x7.0x2.8mm" H 7550 3500 50  0001 C CNN
 F 3 "C408454" H 7550 3500 50  0001 C CNN
 	1    7550 3500
